File: pcb/uniboard/individuals/simhid-g1000_right.sch (EAGLE design)
At the start: 72 parts, among them J4 PCB-INTERCONNECT, J5 ZX62-B-5PA(33)-FULL, J6 2212S, SW27 SLLB510100-HS, SW28 TS-1109S-B-B, SW29 TS-1109S-B-B, SW30 TS-1109S-B-B, SW31 TS-1109S-B-B, SW32 TS-1109S-B-B, SW33 TS-1109S-B-B, SW34 TS-1109S-B-B, U4 STM32F411CCU-ALT, U5 MCP23S18-E/MJ, U6 MCP1703AT-3302E/CB, X1 16MHz/10pF

Commit message: Added non-divisible PCB artwork with the goal of reducing manufacturing costs
Parts:
- added C20: 100nF, gen-discrete3:RCL_C-EUC0402-HS
- J4: value PCB-INTERCONNECT -> PCB-INTERCONNECT-RB; device SimHID-G1000:PCB-INTERCONNECT -> SimHID-G1000:PCB-INTERCONNECT-RB
Connections:
- net +3V3: now also C20.1, U4.VBAT
- net EC7_XA: now also U4.PB10; no longer U4.PB12
- net EC7_XB: now also U4.PB12; no longer U4.PB13
- net EC7_YA: now also U4.PA2; no longer U4.PB2
- net EC7_YB: now also U4.PA4; no longer U4.PB10
- net EC8_A: now also U4.PB13; no longer U4.PB14
- net EC8_B: now also U4.PB14; no longer U4.PB15
- net EC9_XA: now also U4.PB15; no longer U4.PA8
- net EC9_XB: now also U4.PA8; no longer U4.PA9
- net EC9_YA: now also U4.PA9; no longer U4.PA10
- net EC9_YB: now also U4.PA10; no longer U4.PA11
- net EXT1_CS: now also U4.PB2; no longer U4.PB1
- net EXT2_CS: now also U4.PB1; no longer U4.PB0
- net EXT3_CS: now also U4.PB0; no longer U4.PA7
- net GND: now also C20.2, EC5.MH, EC6.MH, EC7.MH, EC9.MH
- net MISO: now also U4.PA6; no longer U4.PA5
- net MOSI: now also U4.PA7; no longer U4.PA4
- net SCLK: now also U4.PA5; no longer U4.PA6
- net USB_D+: now also U4.PA12; no longer U4.PA2
- net USB_D-: now also U4.PA11; no longer U4.PA1
Other:
- moved on the sheet: C8, C9
