File: pcb/uniboard2/individuals/simhid-g1000_left.sch (EAGLE design)
At the start: 33 parts, among them J1 PCB-INTERCONNECT, SW1 SLLB510100-HS, SW10 TS-1109S-B-B, SW11 TS-1109S-B-B, SW12 TS-1109S-B-B, SW13 TS-1109S-B-B, SW14 TS-1109S-B-B, SW2 TS-1109S-B-B, SW3 TS-1109S-B-B, SW4 TS-1109S-B-B, SW5 TS-1109S-B-B, SW6 TS-1109S-B-B, SW7 TS-1109S-B-B, SW8 TS-1109S-B-B, SW9 TS-1109S-B-B, U1 MCP23S17-E, U2 MCP23S17-E

Commit message: Added vertical USB connector versions
Parts:
- J1: value PCB-INTERCONNECT -> PCB-INTERCONNECT-LB; device SimHID-G1000:PCB-INTERCONNECT -> SimHID-G1000:PCB-INTERCONNECT-LB
Changed lines of the file:
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@@
 </classes>
 <parts>
-<part name="J1" library="SimHID-G1000" library_urn="urn:adsk.eagle:library:27646014" deviceset="PCB-INTERCONNECT" device="" package3d_urn="urn:adsk.eagle:package:27646017/2"/>
+<part name="J1" library="SimHID-G1000" library_urn="urn:adsk.eagle:library:27646014" deviceset="PCB-INTERCONNECT" device="-LB" package3d_urn="urn:adsk.eagle:package:41622066/4" value="PCB-INTERCONNECT-LB"/>
 <part name="+3V2" library="supply1" library_urn="urn:adsk.eagle:library:371" deviceset="+3V3" device=""/>
 <part name="GND3" library="supply1" library_urn="urn:adsk.eagle:library:371" deviceset="GND" device=""/>
